File: 0.2/high/ferris.kicad_sch (KiCad schematic)
At the start: 102 parts, among them J1 TYPE-C-31-M-12, K0_0 KEYSW, K0_1 KEYSW, K0_2 KEYSW, K0_3 KEYSW, K0_4 KEYSW, K0_5 KEYSW, K0_6 KEYSW, K0_7 KEYSW, K0_8 KEYSW, K0_9 KEYSW, K1_0 KEYSW, K1_1 KEYSW, K1_2 KEYSW, K1_3 KEYSW, K1_4 KEYSW, K1_5 KEYSW, K1_6 KEYSW, K1_7 KEYSW, K1_8 KEYSW, K1_9 KEYSW, K2_0 KEYSW, K2_1 KEYSW, K2_2 KEYSW, K2_3 KEYSW, K2_4 KEYSW, K2_5 KEYSW, K2_6 KEYSW, K2_7 KEYSW, K2_8 KEYSW, K2_9 KEYSW, K3_3 KEYSW, K3_4 KEYSW, K3_5 KEYSW, K3_6 KEYSW, Q1 PDTC123JT,215, SW1 B3U-1000P, U1 STM32F072CBT6, U2 MCP23017-E/SO, U3 MCP1700T-3302E/TT, U4 SRV05-4

Commit message: bump
Connections:
- net led_data_r: now reaches U2.8 (GPB7)
- net led_data_r: now also K0_5.2 (LED_DIN)
- net led_data_l: now reaches K0_0.2 (LED_DIN)
- net led_data_l: now also U1.13 (PA3)
- no-connect marks 36 -> 34
Changed lines of the file:
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@@
   (no_connect (at 143.51 242.57))
   (no_connect (at 176.53 217.17))
-  (no_connect (at 279.4 207.01))
   (no_connect (at 27.94 217.17))
   (no_connect (at 176.53 219.71))
   (no_connect (at 279.4 227.33))
-  (no_connect (at 176.53 212.09))
   (no_connect (at 279.4 204.47))
   (no_connect (at 143.51 237.49))
@@
     (stroke (width 0) (type default))
   )
+  (wire (pts (xy 222.25 34.29) (xy 226.06 34.29))
+    (stroke (width 0) (type default))
+  )
   (wire (pts (xy 288.29 123.19) (xy 321.31 123.19))
     (stroke (width 0) (type default))
@@
   )
   (wire (pts (xy 58.42 72.39) (xy 58.42 82.55))
+    (stroke (width 0) (type default))
+  )
+  (wire (pts (xy 24.13 34.29) (xy 27.94 34.29))
     (stroke (width 0) (type default))
   )
@@
     (effects (font (size 1.27 1.27)) (justify right bottom))
   )
+  (label "led_data_r" (at 279.4 207.01 0) (fields_autoplaced)
+    (effects (font (size 1.27 1.27)) (justify left bottom))
+  )
   (label "col6" (at 279.4 214.63 0) (fields_autoplaced)
     (effects (font (size 1.27 1.27)) (justify left bottom))
@@
     (effects (font (size 1.27 1.27)) (justify right bottom))
   )
+  (label "led_data_l" (at 24.13 34.29 180) (fields_autoplaced)
+    (effects (font (size 1.27 1.27)) (justify right bottom))
+  )
   (label "D+" (at 176.53 234.95 0) (fields_autoplaced)
     (effects (font (size 1.27 1.27)) (justify left bottom))
@@
     (effects (font (size 1.27 1.27)) (justify right bottom))
   )
+  (label "led_data_r" (at 222.25 34.29 180) (fields_autoplaced)
+    (effects (font (size 1.27 1.27)) (justify right bottom))
+  )
   (label "col4" (at 176.53 240.03 0) (fields_autoplaced)
     (effects (font (size 1.27 1.27)) (justify left bottom))
@@
     (effects (font (size 1.27 1.27)) (justify left bottom))
   )
+  (label "led_data_l" (at 176.53 212.09 0) (fields_autoplaced)
+    (effects (font (size 1.27 1.27)) (justify left bottom))
+  )
